File: ft230x-breakout.kicad_pcb (KiCad board)
At the start: 2 copper layers, 18.2 x 36.4 mm, 20 parts, among them J101 USB_B_Micro, J103 Conn_01x05_Pin, J104 Conn_01x05_Pin, U101 FT230XS

Commit message: Tweak some front silkscreen markings, and add GitHub URL to back silkscreen.
Other:
- board text added: "FT230X Breakout Rev 1.0"
- board text added: "https://github.com/thorpej/ft230x-breakout"
- board text removed: "FT230X Breakout"

Commit message: Correct a silkscreen problem on rev 1.0 of the board: Tx and Rx LED labels were swapped.  Bump rev to 1.1.
Parts:
- D101: value Tx -> Rx
- D102: value Rx -> Tx
Other:
- board text added: "FT230X Breakout Rev 1.1"
- board text removed: "FT230X Breakout Rev 1.0"
Changed lines of the file:
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@@
   (title_block
     (title "FT230X Breakout")
-    (date "2024-07-03")
-    (rev "1.0")
+    (date "2024-07-05")
+    (rev "1.1")
     (company "Copyright (c) 2024 Jason R. Thorpe.  See LICENSE.")
   )
@@
     (descr "LED SMD 0805 (2012 Metric), square (rectangular) end terminal, IPC_7351 nominal, (Body size source: https://docs.google.com/spreadsheets/d/1BsfQQcO9C6DZCsRaXUlFlo91Tg2WpOkGARC1WS5S8t0/edit?usp=sharing), generated with kicad-footprint-generator")
     (tags "LED handsolder")
+    (property "Mouser" "710-150080GS75000")
+    (property "Part" "Wurth 150080GS75000")
     (property "Sheetfile" "ft230x-breakout.kicad_sch")
     (property "Sheetname" "")
@@
         (effects (font (size 0.75 0.75) (thickness 0.1)))
     )
-    (fp_text value "Tx" (at 0 1.65) (layer "F.SilkS")
+    (fp_text value "Rx" (at 0 1.65) (layer "F.SilkS")
         (effects (font (size 1 1) (thickness 0.15)))
     )
@@
     (descr "Capacitor SMD 0805 (2012 Metric), square (rectangular) end terminal, IPC_7351 nominal with elongated pad for handsoldering. (Body size source: IPC-SM-782 page 76, https://www.pcb-3d.com/wordpress/wp-content/uploads/ipc-sm-782a_amendment_1_and_2.pdf, https://docs.google.com/spreadsheets/d/1BsfQQcO9C6DZCsRaXUlFlo91Tg2WpOkGARC1WS5S8t0/edit?usp=sharing), generated with kicad-footprint-generator")
     (tags "capacitor handsolder")
-    (property "Part" "MI0805K400R-10")
+    (property "Mouser" "875-MI0805K400R-10")
+    (property "Part" "Laird MI0805K400R-10")
     (property "Sheetfile" "ft230x-breakout.kicad_sch")
     (property "Sheetname" "")
@@
     (descr "LED SMD 0805 (2012 Metric), square (rectangular) end terminal, IPC_7351 nominal, (Body size source: https://docs.google.com/spreadsheets/d/1BsfQQcO9C6DZCsRaXUlFlo91Tg2WpOkGARC1WS5S8t0/edit?usp=sharing), generated with kicad-footprint-generator")
     (tags "LED handsolder")
+    (property "Mouser" "710-150080RS75000")
+    (property "Part" "Wurth 150080RS75000")
     (property "Sheetfile" "ft230x-breakout.kicad_sch")
     (property "Sheetname" "")
@@
         (effects (font (size 0.75 0.75) (thickness 0.1)))
     )
-    (fp_text value "Rx" (at 0 -1.651) (layer "F.SilkS")
+    (fp_text value "Tx" (at 0 -1.651) (layer "F.SilkS")
         (effects (font (size 1 1) (thickness 0.15)))
     )
@@
     (descr "http://www.molex.com/pdm_docs/sd/1050170001_sd.pdf")
     (tags "Micro-USB SMD Typ-B")
-    (property "Part" "105017-0001")
+    (property "Mouser" "538-105017-0001")
+    (property "Part" "Molex 105017-0001")
     (property "Sheetfile" "ft230x-breakout.kicad_sch")
     (property "Sheetname" "")
@@
     (descr "Tantalum Capacitor SMD AVX-P (2012-15 Metric), IPC_7351 nominal, (Body size from: https://www.vishay.com/docs/40182/tmch.pdf), generated with kicad-footprint-generator")
     (tags "capacitor tantalum")
+    (property "Mouser" "647-F951E475MPAAQ2")
+    (property "Part" "Kyocera AVX F951E475MPAAQ2")
     (property "Sheetfile" "ft230x-breakout.kicad_sch")
     (property "Sheetname" "")
@@
     (effects (font (size 0.75 0.75) (thickness 0.1) italic) (justify left bottom))
   )
-  (gr_text "FT230X Breakout\nRev 1.0" (at 136.4742 101.6254 270) (layer "F.SilkS")
+  (gr_text "FT230X Breakout\nRev 1.1" (at 136.4742 101.6254 270) (layer "F.SilkS")
     (effects (font (size 0.75 0.75) (thickness 0.1) italic) (justify bottom))
   )
